File: Circuitry/HACK Circuit.kicad_sch (KiCad schematic)
At the start: 52 parts, among them J1 Conn_01x02, SW1 SW_Nidec_CAS-120A1, SW10 SW_Push, SW11 SW_Push, SW12 SW_Push, SW13 SW_Push, SW14 SW_Push, SW15 SW_Push, SW16 SW_Push, SW17 SW_Push, SW18 SW_Nidec_CAS-120A1, SW2 SW_Push, SW3 SW_Push, SW4 SW_Push, SW5 SW_Push, SW6 SW_Push, SW7 SW_Push, SW8 SW_Push, SW9 SW_Push

Commit message: Schematic Final Update
Parts:
- removed R12, R13, R14: 330Ω, symbol Device:R_US
- removed SW16, SW17, SW2, SW3, SW4, SW5, SW6, SW7: SW_Push, symbol Switch:SW_Push
- removed SW18: SW_Nidec_CAS-120A1, Button_Switch_SMD:Nidec_Copal_CAS-120A, symbol Switch:SW_Nidec_CAS-120A1
- added D15, D16, D17, D18, D19: LED, symbol Device:LED
- added RV2: 1k, symbol Device:R_Potentiometer
- added U3: ~, symbol HACK Symbols:numpad
Connections:
- net 3V3: now also D10.2 (A), D11.2 (A), D12.2 (A), D13.2 (A), D14.2 (A), D9.2 (A), D15.2 (A), D16.2 (A), D17.2 (A), D19.2 (A), RV2.1
- net GND: now also R10.2, R11.2, R9.2, RV2.3
- net GPIO0: now also U3. (C3)
- net GPIO1: now also U3. (C3)
- net GPIO19: now also U3. (C3); no longer D10.2 (A), D11.2 (A), D9.2 (A)
- net GPIO2: now also U3. (C3)
- net GPIO20: no longer D12.2 (A), D13.2 (A), D14.2 (A)
- net GPIO3: now also U3. (C3)
- net GPIO6: now also U3. (C3)
- net GPIO7: now also U3. (C3)
- net at D7.1 (K), R7.1: now also D13.1 (K)
- net at D5.1 (K), R5.1: now also D15.1 (K)
- net at D8.1 (K), R8.1: now also D12.1 (K)
- net at D14.1 (K): now also D6.1 (K), R6.1
- net at D4.1 (K), R4.1: now also D16.1 (K)
- net GPIO27: now reaches A1.32 (GPIO27_ADC1)
- net GPIO27: now also RV2.2
- net at D1.1 (K), R1.1: now also D19.1 (K)
- net at D3.1 (K), R3.1: now also D17.1 (K)
Other:
- note added: "Filter Dial(GPIO27_ADC)"
- note added: "Key Select (GPIO 0-3/6-7/19)"
- note added: "Power Indication LEDs"
- note added: "SELECTOR"
- note removed: "Flashing LEDs (GPIO 19/20) - Can be more than 3, just proof of plan"
- note removed: "Key Select (GPIO 0/1)"
- note removed: "Loop Station (GPIO 21/22)"
- note removed: "Octave Select (GPIO 6/7)"
- note removed: "Play/Pause"
- note removed: "Record/Reset"
- note removed: "SELECTORS / 2 BTN INPUTS"
- note removed: "Sample/Sound Select (GPIO 2/3)"
- note removed: "Switch Left"
- note removed: "Switch Right"
- moved on the sheet: D10, D11, D2, D3, D4, D5, D6, D7, D8, D9, R10, R11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
